File: hardware/boards/AUXControl.sch (KiCad schematic (older format))
At the start: 0 parts

Commit message: Some more mist schematic edits
Parts:
- added U?: ECP5UM5G-381caBGA, lethalbit:318caBGA, symbol lethalbit:ECP5UM5G-381caBGA
Changed lines of the file:
@@
 Text HLabel 1100 1900 0    50   Input ~ 0
 CLKREQ#
+$Comp
+L lethalbit:ECP5UM5G-381caBGA U?
+U 2 1 5F965335
+P 6050 1700
+F 0 "U?" H 6050 2048 50  0000 C CNN
+F 1 "ECP5UM5G-381caBGA" H 6050 1957 50  0000 C CNN
+F 2 "lethalbit:318caBGA" H 4700 1850 50  0001 C CNN
+F 3 "" H 4700 1850 50  0001 C CNN
+F 4 "Lattice" H 6050 1700 50  0001 C CNN "MFR"
+F 5 "LFE5UM5G-85F-8BG381I" H 6050 1700 50  0001 C CNN "MPN"
+F 6 "220-2112-ND" H 6050 1700 50  0001 C CNN "DIGIKEY_PN"
+	2    6050 1700
+	1    0    0    -1
+$EndComp
 $EndSCHEMATC

Commit message: Lots of small updates, getting values specified for parts, switched the BJT to NFETs
Parts:
- gave numbers to parts that had none: 1
Changed lines of the file:
@@
 $Descr A4 11693 8268
 encoding utf-8
-Sheet 3 11
+Sheet 3 10
 Title ""
 Date ""
@@
 CLKREQ#
 $Comp
-L lethalbit:ECP5UM5G-381caBGA U?
+L lethalbit:ECP5UM5G-381caBGA U1
 U 2 1 5F965335
 P 6050 1700
-F 0 "U?" H 6050 2048 50  0000 C CNN
+F 0 "U1" H 6050 2048 50  0000 C CNN
 F 1 "ECP5UM5G-381caBGA" H 6050 1957 50  0000 C CNN
 F 2 "lethalbit:318caBGA" H 4700 1850 50  0001 C CNN

Commit message: Some strugglebusting on getting the ERC errors cleaned up a bit
Connections:
- no-connect marks 0 -> 37
Changed lines of the file:
@@
 	1    0    0    -1
 $EndComp
+NoConn ~ 5300 1650
+NoConn ~ 5300 1750
+NoConn ~ 5300 1850
+NoConn ~ 5300 1950
+NoConn ~ 5300 2050
+NoConn ~ 5300 2150
+NoConn ~ 5300 2250
+NoConn ~ 5300 2350
+NoConn ~ 5300 2450
+NoConn ~ 5300 2550
+NoConn ~ 5300 2650
+NoConn ~ 5300 2750
+NoConn ~ 5300 2850
+NoConn ~ 5300 2950
+NoConn ~ 6800 1650
+NoConn ~ 6800 1750
+NoConn ~ 6800 1850
+NoConn ~ 6800 1950
+NoConn ~ 6800 2050
+NoConn ~ 6800 2150
+NoConn ~ 6800 2250
+NoConn ~ 6800 2350
+NoConn ~ 6800 2450
+NoConn ~ 6800 2550
+NoConn ~ 6800 2650
+NoConn ~ 6800 2750
+NoConn ~ 6800 2850
+NoConn ~ 1100 750
+NoConn ~ 1100 850
+NoConn ~ 1100 950
+NoConn ~ 1100 1050
+NoConn ~ 1100 1150
+NoConn ~ 1100 1350
+NoConn ~ 1100 1450
+NoConn ~ 1100 1700
+NoConn ~ 1100 1800
+NoConn ~ 1100 1900
 $EndSCHEMATC
