File: hardware/boards/PowerSupply.sch (KiCad schematic (older format))
At the start: 71 parts, among them Q1 Q_NMOS_GSD, Q2 Q_NMOS_GSD, Q3 Q_NMOS_GSD, Q4 Q_NMOS_GSD, Q5 SI7232DN-T1-GE3, U2 ADP5050ACPZ-R7

Commit message: Some strugglebusting on getting the ERC errors cleaned up a bit
Parts:
- R10, R15, R19, R20: value ? -> 10k; MFR (none) -> Vishay Dale; MPN (none) -> RCS060310K0FKEA
- R11: value ? -> 12k1; MFR (none) -> Vishay Dale; MPN (none) -> CRCW060312K1FKEAHP
- R16: value ? -> 8k2; MFR (none) -> Vishay Dale; MPN (none) -> RCS06038K20FKEA
- R17: value ? -> 127k; MFR (none) -> Vishay Dale; MPN (none) -> CRCW0603127KFKEAHP
- R18: value ? -> 4k99; MFR (none) -> Vishay Dale; MPN (none) -> RCS06034K99FKEA
Connections:
- net at U2.46 (COMP_3): now also C10.1, R12.1
- no-connect marks 7 -> 6
Other:
- note removed: "BOT\n"
Changed lines of the file:
@@
 P 6650 2900
 F 0 "R17" H 6709 2946 50  0000 L CNN
-F 1 "?" H 6709 2855 50  0000 L CNN
+F 1 "127k" H 6709 2855 50  0000 L CNN
 F 2 "Resistor_SMD:R_0603_1608Metric" H 6650 2900 50  0001 C CNN
 F 3 "~" H 6650 2900 50  0001 C CNN
+F 4 "Vishay Dale" H 6650 2900 50  0001 C CNN "MFR"
+F 5 "CRCW0603127KFKEAHP" H 6650 2900 50  0001 C CNN "MPN"
 	1    6650 2900
 	1    0    0    -1
@@
 P 6850 3200
 F 0 "R19" V 7046 3200 50  0000 C CNN
-F 1 "?" V 6955 3200 50  0000 C CNN
+F 1 "10k" V 6955 3200 50  0000 C CNN
 F 2 "Resistor_SMD:R_0603_1608Metric" H 6850 3200 50  0001 C CNN
 F 3 "~" H 6850 3200 50  0001 C CNN
+F 4 "Vishay Dale" V 6850 3200 50  0001 C CNN "MFR"
+F 5 "RCS060310K0FKEA" V 6850 3200 50  0001 C CNN "MPN"
 	1    6850 3200
 	0    -1   -1   0
@@
 P 6900 4300
 F 0 "R20" H 6959 4346 50  0000 L CNN
-F 1 "?" H 6959 4255 50  0000 L CNN
+F 1 "10k" H 6959 4255 50  0000 L CNN
 F 2 "Resistor_SMD:R_0603_1608Metric" H 6900 4300 50  0001 C CNN
 F 3 "~" H 6900 4300 50  0001 C CNN
+F 4 "Vishay Dale" H 6900 4300 50  0001 C CNN "MFR"
+F 5 "RCS060310K0FKEA" H 6900 4300 50  0001 C CNN "MPN"
 	1    6900 4300
 	0    1    1    0
@@
 P 6700 4150
 F 0 "R18" H 6759 4196 50  0000 L CNN
-F 1 "?" H 6759 4105 50  0000 L CNN
+F 1 "4k99" H 6759 4105 50  0000 L CNN
 F 2 "Resistor_SMD:R_0603_1608Metric" H 6700 4150 50  0001 C CNN
 F 3 "~" H 6700 4150 50  0001 C CNN
+F 4 "Vishay Dale" H 6700 4150 50  0001 C CNN "MFR"
+F 5 "RCS06034K99FKEA" H 6700 4150 50  0001 C CNN "MPN"
 	1    6700 4150
 	1    0    0    -1
@@
 P 6250 5600
 F 0 "R16" V 6054 5600 50  0000 C CNN
-F 1 "?" V 6145 5600 50  0000 C CNN
+F 1 "8k2" V 6145 5600 50  0000 C CNN
 F 2 "Resistor_SMD:R_0603_1608Metric" H 6250 5600 50  0001 C CNN
 F 3 "~" H 6250 5600 50  0001 C CNN
+F 4 "Vishay Dale" V 6250 5600 50  0001 C CNN "MFR"
+F 5 "RCS06038K20FKEA" V 6250 5600 50  0001 C CNN "MPN"
 	1    6250 5600
 	0    1    1    0
@@
 P 6050 5750
 F 0 "R15" V 5854 5750 50  0000 C CNN
-F 1 "?" V 5945 5750 50  0000 C CNN
+F 1 "10k" V 5945 5750 50  0000 C CNN
 F 2 "Resistor_SMD:R_0603_1608Metric" H 6050 5750 50  0001 C CNN
 F 3 "~" H 6050 5750 50  0001 C CNN
+F 4 "Vishay Dale" V 6050 5750 50  0001 C CNN "MFR"
+F 5 "RCS060310K0FKEA" V 6050 5750 50  0001 C CNN "MPN"
 	1    6050 5750
 	-1   0    0    1
@@
 	5400 6350 5400 6400
 Wire Wire Line
-	5450 5500 5450 6350
+	5450 5450 5450 6350
 Wire Wire Line
 	5450 6350 5400 6350
@@
 P 5250 6000
 F 0 "R11" V 5054 6000 50  0000 C CNN
-F 1 "?" V 5145 6000 50  0000 C CNN
+F 1 "12k1" V 5145 6000 50  0000 C CNN
 F 2 "Resistor_SMD:R_0603_1608Metric" H 5250 6000 50  0001 C CNN
 F 3 "~" H 5250 6000 50  0001 C CNN
+F 4 "Vishay Dale" V 5250 6000 50  0001 C CNN "MFR"
+F 5 "CRCW060312K1FKEAHP" V 5250 6000 50  0001 C CNN "MPN"
 	1    5250 6000
 	0    1    1    0
@@
 P 5100 6200
 F 0 "R10" V 4904 6200 50  0000 C CNN
-F 1 "?" V 4995 6200 50  0000 C CNN
+F 1 "10k" V 4995 6200 50  0000 C CNN
 F 2 "Resistor_SMD:R_0603_1608Metric" H 5100 6200 50  0001 C CNN
 F 3 "~" H 5100 6200 50  0001 C CNN
+F 4 "Vishay Dale" V 5100 6200 50  0001 C CNN "MFR"
+F 5 "RCS060310K0FKEA" V 5100 6200 50  0001 C CNN "MPN"
 	1    5100 6200
 	-1   0    0    1
@@
 	4500 6350 4450 6350
 Connection ~ 4450 6350
-NoConn ~ 2700 1100
-NoConn ~ 2700 1200
 Wire Wire Line
 	3850 5050 3700 5050
@@
 	3700 4750 3700 4900
 Connection ~ 3700 4900
-Text Notes 5100 6250 1    50   ~ 0
-BOT\n
-Text Notes 6050 5850 1    50   ~ 0
-BOT\n
-Text Notes 7000 4300 2    50   ~ 0
-BOT\n
-Text Notes 6950 3200 2    50   ~ 0
-BOT\n
 Wire Wire Line
 	3200 2050 5050 2050
@@
 	1    0    0    -1
 $EndComp
+NoConn ~ 3850 3900
 $EndSCHEMATC

Commit message: Some more ERC cleanup
Connections:
- net 12V0 renamed +12V
Changed lines of the file:
@@
 $EndComp
 NoConn ~ 3850 3900
+Wire Wire Line
+	3700 1000 3700 850
+Connection ~ 3700 1000
+$Comp
+L power:+12V #PWR0119
+U 1 1 5F52525F
+P 3700 850
+F 0 "#PWR0119" H 3700 700 50  0001 C CNN
+F 1 "+12V" H 3715 1023 50  0000 C CNN
+F 2 "" H 3700 850 50  0001 C CNN
+F 3 "" H 3700 850 50  0001 C CNN
+	1    3700 850
+	1    0    0    -1
+$EndComp
 $EndSCHEMATC

Commit message: Switched out the inductor footprints to ones that now have 3d models
Parts:
- L1: footprint Inductor_SMD:L_Coilcraft_XxL4040 -> lethalbit:L_Coilcraft_XxL4040
- L2: footprint Inductor_SMD:L_Coilcraft_XxL4030 -> lethalbit:L_Coilcraft_XxL4030
- L3, L4: footprint Inductor_SMD:L_Coilcraft_XxL4020 -> lethalbit:L_Coilcraft_XxL4020
Changed lines of the file:
@@
 F 0 "L3" H 7200 3615 50  0000 C CNN
 F 1 "3.3uH" H 7200 3524 50  0000 C CNN
-F 2 "Inductor_SMD:L_Coilcraft_XxL4020" H 7200 3400 50  0001 C CNN
+F 2 "lethalbit:L_Coilcraft_XxL4020" H 7200 3400 50  0001 C CNN
 F 3 "~" H 7200 3400 50  0001 C CNN
 F 4 "Coilcraft" H 7200 3400 50  0001 C CNN "MFR"
@@
 F 0 "L2" H 5900 6165 50  0000 C CNN
 F 1 "6.8uH" H 5900 6074 50  0000 C CNN
-F 2 "Inductor_SMD:L_Coilcraft_XxL4030" H 5900 5950 50  0001 C CNN
+F 2 "lethalbit:L_Coilcraft_XxL4030" H 5900 5950 50  0001 C CNN
 F 3 "~" H 5900 5950 50  0001 C CNN
 F 4 "Coilcraft" H 5900 5950 50  0001 C CNN "MFR"
@@
 F 0 "L1" H 4950 6165 50  0000 C CNN
 F 1 "8.2uH" H 4950 6074 50  0000 C CNN
-F 2 "Inductor_SMD:L_Coilcraft_XxL4040" H 4950 5950 50  0001 C CNN
+F 2 "lethalbit:L_Coilcraft_XxL4040" H 4950 5950 50  0001 C CNN
 F 3 "~" H 4950 5950 50  0001 C CNN
 F 4 "Coilcraft" H 4950 5950 50  0001 C CNN "MFR"
@@
 F 0 "L4" H 7200 4715 50  0000 C CNN
 F 1 "4.7uH" H 7200 4624 50  0000 C CNN
-F 2 "Inductor_SMD:L_Coilcraft_XxL4020" H 7200 4500 50  0001 C CNN
+F 2 "lethalbit:L_Coilcraft_XxL4020" H 7200 4500 50  0001 C CNN
 F 3 "~" H 7200 4500 50  0001 C CNN
 F 4 "Coilcraft" H 7200 4500 50  0001 C CNN "MFR"
