File: hardware/boards/lethallink.sch (KiCad schematic (older format))
At the start: 10 parts, among them J1 PCIe-x4

Commit message: In an AHDH fuled stupor I made a bunch of changes, only the last of which I recall, which would be adding fiducials
Parts:
- added FB10: 220 @ 100Mhz, Resistor_SMD:R_0603_1608Metric, symbol Device:Ferrite_Bead_Small
Connections:
- new net IC Power/VBUS: FB10.1
- new net USB3 Interface/VBUS: FB10.2
Changed lines of the file:
@@
 F0 "USB3 Interface" 50
 F1 "USB3Interface.sch" 50
+F2 "VBUS" O L 14700 2350 50
 $EndSheet
 $Sheet
@@
 	9300 3900 10500 3900
 Wire Wire Line
-	8350 4100 9900 4100
-Wire Wire Line
 	10100 4100 10500 4100
-Wire Wire Line
-	8350 3900 9100 3900
 $Sheet
 S 13000 3850 650  500
@@
 F5 "1V2" I L 13000 4000 50
 F6 "1V5" I L 13000 3900 50
+F7 "VBUS" I R 13650 3900 50
 $EndSheet
 $Comp
@@
 Wire Wire Line
 	10300 4000 10300 4450
-Connection ~ 12800 4200
-Wire Wire Line
-	12800 4200 13000 4200
 Connection ~ 12450 4100
 Wire Wire Line
@@
 Wire Wire Line
 	12450 4100 11450 4100
-Wire Wire Line
-	12800 4200 11450 4200
 Wire Wire Line
 	11450 3900 11650 3900
@@
 $EndComp
 Wire Wire Line
-	12800 2550 12800 4200
-Wire Wire Line
-	12450 2550 12450 4100
-Wire Wire Line
-	12050 4000 12050 2550
-Wire Wire Line
-	11650 3900 11650 2550
-Wire Wire Line
 	9700 2550 9700 3450
 Wire Wire Line
@@
 F 3 "" H 11650 2550 50  0001 C CNN
 	1    11650 2550
-	1    0    0    -1
-$EndComp
-$Comp
-L power:+2V5 #PWR?
-U 1 1 5EE12883
-P 12800 2550
-AR Path="/5EDF9F51/5EE12883" Ref="#PWR?"  Part="1"
-AR Path="/5EE12883" Ref="#PWR0108"  Part="1"
-F 0 "#PWR0108" H 12800 2400 50  0001 C CNN
-F 1 "+2V5" H 12815 2723 50  0000 C CNN
-F 2 "" H 12800 2550 50  0001 C CNN
-F 3 "" H 12800 2550 50  0001 C CNN
-	1    12800 2550
 	1    0    0    -1
 $EndComp
@@
 Connection ~ 9100 3900
 Wire Wire Line
-	8350 4000 9500 4000
-Wire Wire Line
 	9500 3450 9500 3700
 Wire Wire Line
@@
 Connection ~ 9500 3700
 Connection ~ 9500 4000
+$Comp
+L Device:Ferrite_Bead_Small FB10
+U 1 1 5F74D6CA
+P 13800 3750
+F 0 "FB10" H 13750 3700 50  0000 R CNN
+F 1 "220 @ 100Mhz" H 13950 3950 50  0001 R CNN
+F 2 "Resistor_SMD:R_0603_1608Metric" V 13730 3750 50  0001 C CNN
+F 3 "~" H 13800 3750 50  0001 C CNN
+F 4 "Murata Electronics" H 13800 3750 50  0001 C CNN "MFR"
+F 5 "BLM18AG221SN1D" H 13800 3750 50  0001 C CNN "MPN"
+	1    13800 3750
+	-1   0    0    1
+$EndComp
+Wire Wire Line
+	13800 3900 13800 3850
+Wire Wire Line
+	13650 3900 13800 3900
+Wire Wire Line
+	13800 3650 13800 2350
+Wire Wire Line
+	13800 2350 14700 2350
+Wire Wire Line
+	12450 2550 12450 4100
+Wire Wire Line
+	12050 4000 12050 2550
+Wire Wire Line
+	11650 3900 11650 2550
+$Comp
+L power:+2V5 #PWR?
+U 1 1 5EE12883
+P 12800 2550
+AR Path="/5EDF9F51/5EE12883" Ref="#PWR?"  Part="1"
+AR Path="/5EE12883" Ref="#PWR0108"  Part="1"
+F 0 "#PWR0108" H 12800 2400 50  0001 C CNN
+F 1 "+2V5" H 12815 2723 50  0000 C CNN
+F 2 "" H 12800 2550 50  0001 C CNN
+F 3 "" H 12800 2550 50  0001 C CNN
+	1    12800 2550
+	1    0    0    -1
+$EndComp
+Wire Wire Line
+	12800 2550 12800 4200
+Wire Wire Line
+	12800 4200 11450 4200
+Wire Wire Line
+	12800 4200 13000 4200
+Connection ~ 12800 4200
+Wire Wire Line
+	8350 4100 9900 4100
+Wire Wire Line
+	8350 4000 9500 4000
+Wire Wire Line
+	8350 3900 9100 3900
 $EndSCHEMATC
