File: hardware/boards/host_card/MechanicalGraphic.sch (KiCad schematic (older format))
At the start: 8 parts

Commit message: Re-routed the USB side of things after adding the ESD diodes for the USB SS lines, still need to add the diode for the normal D+/D- pair
Parts:
- added FID10, FID8, FID9: Fiducial, Fiducial:Fiducial_0.5mm_Mask1mm, symbol Mechanical:Fiducial
Changed lines of the file:
@@
+	1    0    0    -1
+$EndComp
+$Comp
+L Mechanical:Fiducial FID8
+U 1 1 5F41AD6E
+P 1600 3150
+F 0 "FID8" H 1685 3196 50  0000 L CNN
+F 1 "Fiducial" H 1685 3105 50  0000 L CNN
+F 2 "Fiducial:Fiducial_0.5mm_Mask1mm" H 1600 3150 50  0001 C CNN
+F 3 "~" H 1600 3150 50  0001 C CNN
+	1    1600 3150
+	1    0    0    -1
+$EndComp
+$Comp
+L Mechanical:Fiducial FID9
+U 1 1 5F41AD74
+P 1600 3350
+F 0 "FID9" H 1685 3396 50  0000 L CNN
+F 1 "Fiducial" H 1685 3305 50  0000 L CNN
+F 2 "Fiducial:Fiducial_0.5mm_Mask1mm" H 1600 3350 50  0001 C CNN
+F 3 "~" H 1600 3350 50  0001 C CNN
+	1    1600 3350
+	1    0    0    -1
+$EndComp
+$Comp
+L Mechanical:Fiducial FID10
+U 1 1 5F41AD7A
+P 1600 3550
+F 0 "FID10" H 1685 3596 50  0000 L CNN
+F 1 "Fiducial" H 1685 3505 50  0000 L CNN
+F 2 "Fiducial:Fiducial_0.5mm_Mask1mm" H 1600 3550 50  0001 C CNN
+F 3 "~" H 1600 3550 50  0001 C CNN
+	1    1600 3550
 	1    0    0    -1
 $EndComp

Commit message: Added another DDR3 module to expand cache to 8GiB
Parts:
- added FID11: Fiducial, Fiducial:Fiducial_0.5mm_Mask1mm, symbol Mechanical:Fiducial
Changed lines of the file:
@@
+	1    0    0    -1
+$EndComp
+$Comp
+L Mechanical:Fiducial FID11
+U 1 1 5F6F9676
+P 1600 3750
+F 0 "FID11" H 1685 3796 50  0000 L CNN
+F 1 "Fiducial" H 1685 3705 50  0000 L CNN
+F 2 "Fiducial:Fiducial_0.5mm_Mask1mm" H 1600 3750 50  0001 C CNN
+F 3 "~" H 1600 3750 50  0001 C CNN
+	1    1600 3750
 	1    0    0    -1
 $EndComp

Commit message: Minor cleanup and added some notes
Parts:
- added FID12: Fiducial, Fiducial:Fiducial_0.5mm_Mask1mm, symbol Mechanical:Fiducial
Changed lines of the file:
@@
+	1    0    0    -1
+$EndComp
+$Comp
+L Mechanical:Fiducial FID12
+U 1 1 600FE625
+P 1600 3950
+F 0 "FID12" H 1685 3996 50  0000 L CNN
+F 1 "Fiducial" H 1685 3905 50  0000 L CNN
+F 2 "Fiducial:Fiducial_0.5mm_Mask1mm" H 1600 3950 50  0001 C CNN
+F 3 "~" H 1600 3950 50  0001 C CNN
+	1    1600 3950
 	1    0    0    -1
 $EndComp
