File: hardware/boards/host_card/DebugInterface.sch (KiCad schematic (older format))
At the start: 2 parts, among them J6 SODIMM_260, U1 ECP5UM5G-381caBGA

Commit message: Updated the generic SODIMM part footprint to use the new Debug Module footprint
Parts:
- J6: footprint lethalbit-connectors:TE_SODIMM_260 -> lethalbit-connectors:lethallink_Debug_Module_Mount
Changed lines of the file:
@@
 F 0 "J6" H 10100 2425 50  0000 C CNN
 F 1 "SODIMM_260" H 10100 2334 50  0000 C CNN
-F 2 "lethalbit-connectors:TE_SODIMM_260" H 10100 2200 50  0001 C CNN
+F 2 "lethalbit-connectors:lethallink_Debug_Module_Mount" H 10100 2200 50  0001 C CNN
 F 3 "https://www.te.com/commerce/DocumentDelivery/DDEController?Action=srchrtrv&DocNm=2309413&DocType=Customer+Drawing&DocLang=English" H 10100 2200 50  0001 C CNN
 F 4 "TE Connectivity AMP Connectors" H 10100 1850 50  0001 C CNN "MFR"
@@
 F 0 "J6" H 10100 6025 50  0000 C CNN
 F 1 "SODIMM_260" H 10100 5934 50  0000 C CNN
-F 2 "lethalbit-connectors:TE_SODIMM_260" H 10100 5800 50  0001 C CNN
+F 2 "lethalbit-connectors:lethallink_Debug_Module_Mount" H 10100 5800 50  0001 C CNN
 F 3 "https://www.te.com/commerce/DocumentDelivery/DDEController?Action=srchrtrv&DocNm=2309413&DocType=Customer+Drawing&DocLang=English" H 10100 5800 50  0001 C CNN
 F 4 "TE connectivity AMP Connectors" H 10100 5450 50  0001 C CNN "MFR"

Commit message: Some updates with the debug module interface
Parts:
- J6: footprint lethalbit-connectors:lethallink_Debug_Module_Mount -> lethallink:lethallink_debug_module_mount
Changed lines of the file:
@@
 F 0 "J6" H 10100 2425 50  0000 C CNN
 F 1 "SODIMM_260" H 10100 2334 50  0000 C CNN
-F 2 "lethalbit-connectors:lethallink_Debug_Module_Mount" H 10100 2200 50  0001 C CNN
+F 2 "lethallink:lethallink_debug_module_mount" H 10100 2200 50  0001 C CNN
 F 3 "https://www.te.com/commerce/DocumentDelivery/DDEController?Action=srchrtrv&DocNm=2309413&DocType=Customer+Drawing&DocLang=English" H 10100 2200 50  0001 C CNN
 F 4 "TE Connectivity AMP Connectors" H 10100 1850 50  0001 C CNN "MFR"
@@
 F 0 "J6" H 10100 6025 50  0000 C CNN
 F 1 "SODIMM_260" H 10100 5934 50  0000 C CNN
-F 2 "lethalbit-connectors:lethallink_Debug_Module_Mount" H 10100 5800 50  0001 C CNN
+F 2 "lethallink:lethallink_debug_module_mount" H 10100 5800 50  0001 C CNN
 F 3 "https://www.te.com/commerce/DocumentDelivery/DDEController?Action=srchrtrv&DocNm=2309413&DocType=Customer+Drawing&DocLang=English" H 10100 5800 50  0001 C CNN
 F 4 "TE connectivity AMP Connectors" H 10100 5450 50  0001 C CNN "MFR"

Commit message: Fixed  / updated the ECP5 symbol for the ECP5UM5G-85K
Parts:
- U1: symbol lethalbit:ECP5UM5G-381caBGA -> lethalbit:LFE5UM5G-85F-8BG381I
Changed lines of the file:
@@
 Comment4 ""
 $EndDescr
-NoConn ~ 4950 3100
-NoConn ~ 4950 3200
-NoConn ~ 4950 3300
-NoConn ~ 4950 3400
-NoConn ~ 4950 3500
-NoConn ~ 4950 3600
-NoConn ~ 4950 3700
-NoConn ~ 4950 3800
-NoConn ~ 4950 3900
-NoConn ~ 4950 4000
-NoConn ~ 4950 4100
-NoConn ~ 4950 4200
-NoConn ~ 4950 4300
-NoConn ~ 4950 4400
-NoConn ~ 4950 4500
-NoConn ~ 4950 4600
-NoConn ~ 4950 4700
-NoConn ~ 6750 4500
-NoConn ~ 6750 4400
-NoConn ~ 6750 4300
-NoConn ~ 6750 4200
-NoConn ~ 6750 4100
-NoConn ~ 6750 4000
-NoConn ~ 6750 3900
-NoConn ~ 6750 3800
-NoConn ~ 6750 3700
-NoConn ~ 6750 3600
-NoConn ~ 6750 3500
-NoConn ~ 6750 3400
-NoConn ~ 6750 3300
-NoConn ~ 6750 3200
-NoConn ~ 6750 3100
+NoConn ~ 5350 3100
+NoConn ~ 5350 3200
+NoConn ~ 5350 3300
+NoConn ~ 5350 3400
+NoConn ~ 5350 3500
+NoConn ~ 5350 3600
+NoConn ~ 5350 3700
+NoConn ~ 5350 3800
+NoConn ~ 5350 3900
+NoConn ~ 5350 4000
+NoConn ~ 5350 4100
+NoConn ~ 5350 4200
+NoConn ~ 5350 4300
+NoConn ~ 5350 4400
+NoConn ~ 5350 4500
+NoConn ~ 5350 4600
+NoConn ~ 5350 4700
+NoConn ~ 6350 4500
+NoConn ~ 6350 4400
+NoConn ~ 6350 4300
+NoConn ~ 6350 4200
+NoConn ~ 6350 4100
+NoConn ~ 6350 4000
+NoConn ~ 6350 3900
+NoConn ~ 6350 3800
+NoConn ~ 6350 3700
+NoConn ~ 6350 3600
+NoConn ~ 6350 3500
+NoConn ~ 6350 3400
+NoConn ~ 6350 3300
+NoConn ~ 6350 3200
+NoConn ~ 6350 3100
 $Comp
-L lethalbit:ECP5UM5G-381caBGA U?
+L lethalbit:LFE5UM5G-85F-8BG381I U?
 U 3 1 610DED19
 P 5850 3150
@@
 	1    0    0    -1
 $EndComp
-NoConn ~ 6750 4600
+NoConn ~ 6350 4600
 $Comp
 L lethalbit:SODIMM_260 J6
