File: hardware/boards/host_card/BootConfig.sch (KiCad schematic (older format))
At the start: 37 parts, among them J3 Conn_02x05_Odd_Even, J4 Conn_02x04_Odd_Even, Q6 Q_NMOS_GSD, Q7 Q_NMOS_GSD, SW1 SW_DIP_x03, SW2 RESET, U1 ECP5UM5G-381caBGA, U3 CYUSB3014, U5 128MiB, Y1 19.2MHz

Commit message: Added a fiducial to for U7. Changed the two pin-headers to the keyd  samtec connectors. Some other misc updates
Parts:
- J4: footprint Connector_PinHeader_1.27mm:PinHeader_2x05_P1.27mm_Vertical -> lethalbit-connectors:FTSH-105-01-L-DV-K-TR
Changed lines of the file:
@@
 F 0 "J4" H 6200 2817 50  0000 C CNN
 F 1 "Conn_02x04_Odd_Even" H 6200 2726 50  0000 C CNN
-F 2 "Connector_PinHeader_1.27mm:PinHeader_2x05_P1.27mm_Vertical" H 6150 2400 50  0001 C CNN
+F 2 "lethalbit-connectors:FTSH-105-01-L-DV-K-TR" H 6150 2400 50  0001 C CNN
 F 3 "~" H 6150 2400 50  0001 C CNN
 	1    6150 2400

Commit message: Added a pin-header for the FPGA SPI flash lines to allow for the USB PHY to do a DFU update of the gateware when closed
Parts:
- added J7: Conn_02x04_Odd_Even, Connector_PinHeader_2.54mm:PinHeader_2x04_P2.54mm_Vertical, symbol Connector_Generic:Conn_02x04_Odd_Even
Connections:
- net 3V3: now also J4.4 (Pin_4); no longer J4.3 (Pin_3)
- net GND: now also J4.3 (Pin_3); no longer J4.4 (Pin_4)
- net ~INIT: now also J4.1 (Pin_1); no longer J4.2 (Pin_2)
- net ~RESET: now also J4.2 (Pin_2); no longer J4.1 (Pin_1)
- net at U1.R2 (PB15A/HOLDN/DI/BUSY/CSSPIN/CEN), U5.1 (~CS): now also J4.10 (Pin_10), J7.2 (Pin_2); no longer J4.9 (Pin_9)
- net at R44.2, U1.W2 (PB11B/D0/MOSI/IO2), U5.2 (DO/IO1): now also J4.8 (Pin_8), J7.4 (Pin_4); no longer J4.7 (Pin_7)
- net at R43.2, U1.Y2 (PB9B/D2/IO2), U5.3 (~WP~/IO2): now also J4.6 (Pin_6); no longer J4.5 (Pin_5)
- net at R46.2, U1.V2 (PB11A/D1/MISO/IO1), U5.5 (DI/IO0): now also J4.5 (Pin_5), J7.6 (Pin_6); no longer J4.6 (Pin_6)
- net at R42.1, U5.6 (CLK): now also J4.7 (Pin_7), J7.8 (Pin_8); no longer J4.8 (Pin_8)
- net at R45.2, U1.W1 (PB8A/D3/IO3), U5.7 (~HOLD~/IO3): now also J4.9 (Pin_9); no longer J4.10 (Pin_10)
- new net FPGA_CLK: J7.7 (Pin_7)
- new net FPGA_DI: J7.5 (Pin_5)
- new net FPGA_DO: J7.3 (Pin_3)
- new net ~FPGA_CS: J7.1 (Pin_1)
Other:
- note added: "FPGA SPI flash USB PHY jumper.\n\nClose to enable DFU for gateware"
- note added: "SPI Flash Pinout\n01 - ~INIT~\n02 - ~PROGRAM~\n03 - GND\n04 - 3v3\n05 - DI/IO0\n06 - ~WP~/IO2\n07 - CLK\n08 - DO/IO1\n09 - ~HOLD~/IO3\n10 - ~CS~\n"
- note removed: "SPI Flash Pinout\n01 - ~PROGRAM~\n02 - ~INIT~\n03 - 3v3\n04 - GND\n05 - ~WP~/IO2\n06 - DI/IO0\n07 - DO/IO1\n08 - CLK\n09 - ~CS~\n10 - ~HOLD~/IO3\n"
Changed lines of the file:
@@
 L Connector_Generic:Conn_02x05_Odd_Even J4
 U 1 1 60CB5062
-P 6150 2400
-F 0 "J4" H 6200 2817 50  0000 C CNN
-F 1 "Conn_02x04_Odd_Even" H 6200 2726 50  0000 C CNN
-F 2 "lethalbit-connectors:FTSH-105-01-L-DV-K-TR" H 6150 2400 50  0001 C CNN
-F 3 "~" H 6150 2400 50  0001 C CNN
-	1    6150 2400
-	1    0    0    -1
+P 6250 2400
+F 0 "J4" H 6300 2817 50  0000 C CNN
+F 1 "Conn_02x04_Odd_Even" H 6300 2726 50  0000 C CNN
+F 2 "lethalbit-connectors:FTSH-105-01-L-DV-K-TR" H 6250 2400 50  0001 C CNN
+F 3 "~" H 6250 2400 50  0001 C CNN
+	1    6250 2400
+	-1   0    0    -1
 $EndComp
 Wire Wire Line
@@
 	8100 4650 8450 4650
 Text Notes 5600 1850 0    50   ~ 0
-SPI Flash Pinout\n01 - ~PROGRAM~\n02 - ~INIT~\n03 - 3v3\n04 - GND\n05 - ~WP~/IO2\n06 - DI/IO0\n07 - DO/IO1\n08 - CLK\n09 - ~CS~\n10 - ~HOLD~/IO3\n
+SPI Flash Pinout\n01 - ~INIT~\n02 - ~PROGRAM~\n03 - GND\n04 - 3v3\n05 - DI/IO0\n06 - ~WP~/IO2\n07 - CLK\n08 - DO/IO1\n09 - ~HOLD~/IO3\n10 - ~CS~\n
 Text HLabel 7900 7400 0    39   Input ~ 0
 ~PHY_RESET
@@
 	4900 3400 4900 5450
 Wire Wire Line
-	7400 3500 7400 4150
+	7400 3500 7400 3700
 Wire Wire Line
 	4700 3950 4700 5050
@@
 Text Label 7400 4750 0    50   ~ 0
 DONE
+Text HLabel 3500 3400 0    39   Input ~ 0
+~FPGA_CS
+Text HLabel 3500 3500 0    39   Input ~ 0
+FPGA_DO
+Text HLabel 3500 3600 0    39   Input ~ 0
+FPGA_DI
+Text HLabel 3500 3700 0    39   Input ~ 0
+FPGA_CLK
+$Comp
+L Connector_Generic:Conn_02x04_Odd_Even J7
+U 1 1 5FC575A5
+P 3900 3500
+F 0 "J7" H 3950 3817 50  0000 C CNN
+F 1 "Conn_02x04_Odd_Even" H 3950 3726 50  0000 C CNN
+F 2 "Connector_PinHeader_2.54mm:PinHeader_2x04_P2.54mm_Vertical" H 3900 3500 50  0001 C CNN
+F 3 "~" H 3900 3500 50  0001 C CNN
+	1    3900 3500
+	1    0    0    -1
+$EndComp
+Wire Wire Line
+	3500 3400 3700 3400
+Wire Wire Line
+	3500 3500 3700 3500
+Wire Wire Line
+	3500 3600 3700 3600
+Wire Wire Line
+	3500 3700 3700 3700
+Wire Wire Line
+	4200 3400 4900 3400
+Connection ~ 4900 3400
+Wire Wire Line
+	4200 3500 4750 3500
+Connection ~ 4750 3500
+Wire Wire Line
+	4200 3600 4700 3600
+Wire Wire Line
+	4700 3600 4700 3950
+Connection ~ 4700 3950
+Wire Wire Line
+	4200 3700 7400 3700
+Connection ~ 7400 3700
+Wire Wire Line
+	7400 3700 7400 4150
+Text Notes 3300 3050 0    50   ~ 0
+FPGA SPI flash USB PHY jumper.\n\nClose to enable DFU for gateware
 $EndSCHEMATC

Commit message: Started poking the SPI flash for the USB PHY
Parts:
- R55: footprint Resistor_SMD:R_0603_1608Metric -> Resistor_SMD:R_0402_1005Metric; MPN CRCW06031K00FKEAHP -> RCS04021K00FKED
Changed lines of the file:
@@
 F 0 "R55" H 8859 6596 50  0000 L CNN
 F 1 "1k" H 8859 6505 50  0000 L CNN
-F 2 "Resistor_SMD:R_0603_1608Metric" H 8800 6550 50  0001 C CNN
+F 2 "Resistor_SMD:R_0402_1005Metric" H 8800 6550 50  0001 C CNN
 F 3 "~" H 8800 6550 50  0001 C CNN
 F 4 "Vishay Dale" H 8800 6550 50  0001 C CNN "MFR"
-F 5 "CRCW06031K00FKEAHP" H 8800 6550 50  0001 C CNN "MPN"
+F 5 "RCS04021K00FKED" H 8800 6550 50  0001 C CNN "MPN"
 	1    8800 6550
 	1    0    0    -1

Commit message: Fixed  / updated the ECP5 symbol for the ECP5UM5G-85K
Parts:
- U1: symbol lethalbit:ECP5UM5G-381caBGA -> lethalbit:LFE5UM5G-85F-8BG381I
Changed lines of the file:
@@
 Comment4 ""
 $EndDescr
-$Comp
-L lethalbit:ECP5UM5G-381caBGA U?
-U 8 1 5F21A733
-P 6200 4500
-AR Path="/5F21A733" Ref="U?"  Part="8"
-AR Path="/5EF66188/5F21A733" Ref="U?"  Part="8"
-AR Path="/5EF66251/5F21A733" Ref="U1"  Part="8"
-F 0 "U1" H 6250 4848 50  0000 C CNN
-F 1 "ECP5UM5G-381caBGA" H 6250 4757 50  0000 C CNN
-F 2 "lethalbit:318caBGA" H 4850 4650 50  0001 C CNN
-F 3 "" H 4850 4650 50  0001 C CNN
-F 4 "Lattice" H 6200 4500 50  0001 C CNN "MFR"
-F 5 "LFE5UM5G-85F-8BG381I" H 6200 4500 50  0001 C CNN "MPN"
-F 6 "220-2112-ND" H 6200 4500 50  0001 C CNN "DIGIKEY_PN"
-	8    6200 4500
-	1    0    0    -1
-$EndComp
 NoConn ~ 5200 4450
 NoConn ~ 5200 5250
@@
 Text Notes 3300 3050 0    50   ~ 0
 FPGA SPI flash USB PHY jumper.\n\nClose to enable DFU for gateware
+$Comp
+L lethalbit:LFE5UM5G-85F-8BG381I U?
+U 8 1 5F21A733
+P 6200 4500
+AR Path="/5F21A733" Ref="U?"  Part="8"
+AR Path="/5EF66188/5F21A733" Ref="U?"  Part="8"
+AR Path="/5EF66251/5F21A733" Ref="U1"  Part="8"
+F 0 "U1" H 6250 4848 50  0000 C CNN
+F 1 "ECP5UM5G-381caBGA" H 6250 4757 50  0000 C CNN
+F 2 "lethalbit:318caBGA" H 4850 4650 50  0001 C CNN
+F 3 "" H 4850 4650 50  0001 C CNN
+F 4 "Lattice" H 6200 4500 50  0001 C CNN "MFR"
+F 5 "LFE5UM5G-85F-8BG381I" H 6200 4500 50  0001 C CNN "MPN"
+F 6 "220-2112-ND" H 6200 4500 50  0001 C CNN "DIGIKEY_PN"
+	8    6200 4500
+	1    0    0    -1
+$EndComp
 $EndSCHEMATC

Commit message: Swizzled the pins on the PHY bus to make routing to the FPGA nicer, also did the initial bus routing
Parts:
- removed R36, R8: 1k, Resistor_SMD:R_0603_1608Metric, symbol Device:R_Small
- removed SW1: SW_DIP_x03, Button_Switch_SMD:SW_DIP_SPSTx04_Slide_6.7x11.72mm_W8.61mm_P2.54mm_LowProfile, symbol Switch:SW_DIP_x04
Connections:
- net GND: now also U1.R4 (CFG_2), U1.U4 (CFG_0)
- no-connect marks 12 -> 10
Other:
- note added: "CFG[0..2] should be\n0 1 0 for SPI primary."
- note removed: "CFG[0..2] should be\n0 1 0 for SPI master."
- note removed: "This should just be replaced with the proper\npull-ups/downs to statically configure,\nbut for rev 0 lets let it be configurable."
Changed lines of the file:
@@
 NoConn ~ 5200 5550
 Wire Wire Line
-	7300 4950 9800 4950
-Wire Wire Line
 	7300 5050 9550 5050
-Wire Wire Line
-	7300 5150 9300 5150
 $Comp
 L power:GND #PWR0120
 U 1 1 5F051E7C
-P 10600 5250
-F 0 "#PWR0120" H 10600 5000 50  0001 C CNN
-F 1 "GND" H 10605 5077 50  0000 C CNN
-F 2 "" H 10600 5250 50  0001 C CNN
-F 3 "" H 10600 5250 50  0001 C CNN
-	1    10600 5250
-	1    0    0    -1
-$EndComp
-Wire Wire Line
-	10500 4950 10600 4950
-Wire Wire Line
-	10600 4950 10600 5050
-Wire Wire Line
-	10500 5050 10600 5050
-Connection ~ 10600 5050
-Wire Wire Line
-	10600 5050 10600 5150
-Wire Wire Line
-	10500 5150 10600 5150
-Connection ~ 10600 5150
-Wire Wire Line
-	10600 5150 10600 5250
-$Comp
-L Device:R_Small R36
-U 1 1 5F07FA1E
-P 9800 4500
-F 0 "R36" H 9859 4546 50  0000 L CNN
-F 1 "1k" H 9859 4455 50  0000 L CNN
-F 2 "Resistor_SMD:R_0603_1608Metric" H 9800 4500 50  0001 C CNN
-F 3 "~" H 9800 4500 50  0001 C CNN
-F 4 "Vishay Dale" H 9800 4500 50  0001 C CNN "MFR"
-F 5 "CRCW06031K00FKEAHP" H 9800 4500 50  0001 C CNN "MPN"
-	1    9800 4500
-	1    0    0    -1
-$EndComp
+P 10000 5250
+F 0 "#PWR0120" H 10000 5000 50  0001 C CNN
+F 1 "GND" H 10005 5077 50  0000 C CNN
+F 2 "" H 10000 5250 50  0001 C CNN
+F 3 "" H 10000 5250 50  0001 C CNN
+	1    10000 5250
+	1    0    0    -1
+$EndComp
+Connection ~ 10000 5150
+Wire Wire Line
+	10000 5150 10000 5250
 $Comp
 L Device:R_Small R9
@@
 	1    0    0    -1
 $EndComp
-$Comp
-L Device:R_Small R8
-U 1 1 5F08AA7C
-P 9300 4500
-F 0 "R8" H 9359 4546 50  0000 L CNN
-F 1 "1k" H 9359 4455 50  0000 L CNN
-F 2 "Resistor_SMD:R_0603_1608Metric" H 9300 4500 50  0001 C CNN
-F 3 "~" H 9300 4500 50  0001 C CNN
-F 4 "Vishay Dale" H 9300 4500 50  0001 C CNN "MFR"
-F 5 "CRCW06031K00FKEAHP" H 9300 4500 50  0001 C CNN "MPN"
-	1    9300 4500
-	1    0    0    -1
-$EndComp
-Wire Wire Line
-	9300 4600 9300 5150
-Connection ~ 9300 5150
-Wire Wire Line
-	9300 5150 9900 5150
 Wire Wire Line
 	9550 4600 9550 5050
-Connection ~ 9550 5050
-Wire Wire Line
-	9550 5050 9900 5050
-Wire Wire Line
-	9800 4600 9800 4950
-Connection ~ 9800 4950
-Wire Wire Line
-	9800 4950 9900 4950
-Wire Wire Line
-	9300 4400 9300 4250
-Wire Wire Line
-	9300 4250 9550 4250
-Wire Wire Line
-	9800 4250 9800 4400
 Wire Wire Line
 	9550 4400 9550 4250
 Connection ~ 9550 4250
-Wire Wire Line
-	9550 4250 9800 4250
 Wire Wire Line
 	9550 4250 9550 4150
@@
 Wire Wire Line
 	7250 6600 7600 6600
-$Comp
-L Switch:SW_DIP_x04 SW1
-U 1 1 5EF8C546
-P 10200 5050
-F 0 "SW1" H 10200 5517 50  0000 C CNN
-F 1 "SW_DIP_x03" H 10200 5426 50  0000 C CNN
-F 2 "Button_Switch_SMD:SW_DIP_SPSTx04_Slide_6.7x11.72mm_W8.61mm_P2.54mm_LowProfile" H 10200 5050 50  0001 C CNN
-F 3 "~" H 10200 5050 50  0001 C CNN
-F 4 "Würth Elektronik" H 10200 5050 50  0001 C CNN "MFR"
-F 5 "418121270804" H 10200 5050 50  0001 C CNN "MPN"
-	1    10200 5050
-	1    0    0    -1
-$EndComp
-NoConn ~ 10500 4850
-NoConn ~ 9900 4850
 Wire Wire Line
 	7400 4550 7400 4350
@@
 Wire Wire Line
 	5000 3600 5550 3600
-Text Notes 10750 4600 0    50   ~ 0
-CFG[0..2] should be\n0 1 0 for SPI master.
-Text Notes 10750 4950 0    50   ~ 0
-This should just be replaced with the proper\npull-ups/downs to statically configure,\nbut for rev 0 lets let it be configurable.
+Text Notes 9700 4850 0    50   ~ 0
+CFG[0..2] should be\n0 1 0 for SPI primary.
 $Comp
 L power:GND #PWR0128
@@
 Wire Wire Line
 	8450 4300 8450 4250
-Wire Wire Line
-	8450 4250 9300 4250
-Connection ~ 9300 4250
 $Comp
 L Device:LED D10
@@
 	1    0    0    -1
 $EndComp
+Wire Wire Line
+	8450 4250 9550 4250
+Wire Wire Line
+	10000 4950 10000 5150
+Wire Wire Line
+	7300 4950 10000 4950
+Wire Wire Line
+	7300 5150 10000 5150
 $EndSCHEMATC

Commit message: Lots of updates from a while ago, don't recall what's changed
Parts:
- J4: MFR (none) -> Samtec; MPN (none) -> FTSH-105-01-L-DV-K-TR
Connections:
- net TDO: now also J3.6 (Pin_6), R40.2, U3.C10 (TDO); no longer U1.V4 (TDO), U3.E7 (TDI)
- new net FPGA_TDO: U1.V4 (TDO), U3.E7 (TDI)
Changed lines of the file:
@@
 F 2 "lethalbit-connectors:FTSH-105-01-L-DV-K-TR" H 6250 2400 50  0001 C CNN
 F 3 "~" H 6250 2400 50  0001 C CNN
+F 4 "Samtec" H 6250 2400 50  0001 C CNN "MFR"
+F 5 "FTSH-105-01-L-DV-K-TR" H 6250 2400 50  0001 C CNN "MPN"
 	1    6250 2400
 	-1   0    0    -1
@@
 	4800 3600 4800 4950
 Text Label 7350 5350 0    50   ~ 0
-TDO
+FPGA_TDO
 Text Label 7350 5450 0    50   ~ 0
 TCK
@@
 Wire Wire Line
 	7300 5150 10000 5150
+Text Label 8800 5950 0    50   ~ 0
+TDO
 $EndSCHEMATC

Commit message: Broke out the DDR3 modules and added the 0.75V LDO for the VREFCA and VREFDQ lines for each of the DDR3 modules
Connections:
- net XTAL+: now reaches C56.2, U3.C6 (XTAL_IN), Y1.3
- net XTAL-: now reaches C55.2, U3.C7 (XTAL_OUT), Y1.1
- net DONE renamed FPGA_DONE
Changed lines of the file:
@@
 Wire Wire Line
 	8550 3350 9150 3350
-Wire Wire Line
-	9150 3350 9150 4350
 Connection ~ 9150 4650
 $Comp
@@
 Text Label 8800 5950 0    50   ~ 0
 TDO
+Wire Wire Line
+	9150 3350 9150 4350
+Text HLabel 7800 4850 0    39   Output ~ 0
+FPGA_DONE
+Wire Wire Line
+	7800 4850 8100 4850
+Text Label 8100 4850 2    50   ~ 0
+DONE
+Text Label 10350 6200 0    50   ~ 0
+XTAL+
+Text Label 10350 6300 0    50   ~ 0
+XTAL-
 $EndSCHEMATC
