File: hardware/boards/host_card/PowerSupply.sch (KiCad schematic (older format))
At the start: 78 parts, among them Q1 Q_NMOS_GSD, Q2 Q_NMOS_GSD, Q3 Q_NMOS_GSD, Q4 Q_NMOS_GSD, Q5 SI7232DN-T1-GE3, U2 ADP5050ACPZ-R7

Commit message: Broke out the DDR3 modules and added the 0.75V LDO for the VREFCA and VREFDQ lines for each of the DDR3 modules
Parts:
- R26: Field5 CRCW06034K22FKEAHP -> (none); MPN (none) -> CRCW06034K22FKEAHP
Changed lines of the file:
@@
 F 3 "~" H 9950 6850 50  0001 C CNN
 F 4 "Vishay Dale" V 9950 6850 50  0001 C CNN "MFR"
-F 5 "CRCW06034K22FKEAHP" V 9950 6850 50  0001 C CNN "Field5"
+F 5 "CRCW06034K22FKEAHP" V 9950 6850 50  0001 C CNN "MPN"
 	1    9950 6850
 	0    1    1    0
